File: sinobit.sch (EAGLE design)
At the start: 253 parts, among them J1 TWIG_2.0, J2 TWIG_2.0, U1 SPX3819, U10 16MHZ2520, U6 IC_NRF51822_MODULE, U8 HT1632C_QFP52, U9 16MHZ2520

Commit message: sinobit-V1.0
Parts:
- C33: value 22uF -> 10uF
- R26, R28, R29, R30, R31, R32: value 3.3M -> 2M
- R33: value 525K -> 510k
- renumbered U$13 to U14, U$4 to U16, U$6 to U11, U$7 to U12
Connections:
- removed net N$7: R30.2, U$51.P$1, U6.P0.03
- removed net P0.8: U$12.9, U6.P0.08
- new net P0.3: R30.2, U$12.25, U$51.P$1, U6.P0.03
- net 3.3V: now also U$12.13; no longer U$12.14
- net 8653_INT2: no longer U$12.2
- net BTN_A: now also U$12.4
- net BTN_B: now also U$12.8; no longer U$12.3
- net GND: now also U$12.14; no longer U$12.13
- net MISO: now also U$12.17; no longer U$12.4
- net MOSI: now also U$12.10
- net P0.10: now also U$12.6; no longer U$12.10
- net P0.11: now also U$12.5; no longer U$12.17
- net P0.12: now also U$12.22; no longer U$12.11
- net P0.13: now also U$12.15; no longer U$12.16
- net P0.14: no longer U$12.12
- net P0.15: no longer U$12.15
- net P0.16: now also U$12.16
- net P0.18: now also U$12.21
- net P0.2/RX: now also U$12.2; no longer U$12.23
- net P0.20: now also U$12.18; no longer U$12.5
- net P0.4: now also U$12.3; no longer U$12.22
- net P0.5: now also U$12.23; no longer U$12.21
- net P0.6: now also U$12.19; no longer U$12.8
- net P0.7: no longer U$12.19
- net P0.9: no longer U$12.18
- net SCK: now also U$12.9
- net SCL: now also U$12.11; no longer U$12.25
- net SDA: now also U$12.12
- net TGT_NRESET: no longer U$12.6
Other:
- note added: "Creator :"
- note added: "Elecrow"
- note added: "Naomi Wu"
- note added: "Sheet :"
- note removed: "Creator:"
- note removed: "Engle&Keen"
- note removed: "Naomi"
- note removed: "sheet :"
